File: _autosave-ESP32_WROOM_32E_msd.kicad_sch (KiCad schematic)
At the start: 27 parts, among them J10 7.5V, J9 Motor_Driver, SW1 SW_SPDT, U2 MCP2561-E-SN

Commit message: complete ver2
Parts:
- SW1: footprint Connector_PinHeader_2.54mm:PinHeader_1x03_P2.54mm_Vertical_SMD_Pin1Right -> Connector_PinHeader_2.54mm:PinHeader_1x03_P2.54mm_Vertical
Changed lines of the file:
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@@
 			)
 		)
-		(property "Footprint" "Connector_PinHeader_2.54mm:PinHeader_1x03_P2.54mm_Vertical_SMD_Pin1Right"
+		(property "Footprint" "Connector_PinHeader_2.54mm:PinHeader_1x03_P2.54mm_Vertical"
 			(at 67.31 160.02 0)
 			(effects
